Commit message: restructured pc files into week folders

File: src/Week04/hyper_pupper_complete/urdf/leg.urdf.xacro (robot description, xacro)
@@ -7,5 +7,5 @@
             <xacro:property name="upper_leg_to_lower_leg" value="${upper_leg_to_lower_leg_distance}" />
             <xacro:property name="hip_mesh_path" value="package://hyper_pupper_complete/meshes/${leg}_hip.stl" />
-            <xacro:property name="upper_leg_mesh_path" value="package://hyper_pupper_complete/meshes/${leg}_upper_leg.stl" />
+            <xacro:property name="upper_leg_mesh_path" value="package://hyper_pupper_complete/meshes/${leg}_lower_leg.stl" />
             <xacro:property name="lower_leg_mesh_path" value="package://hyper_pupper_complete/meshes/${leg}_lower_leg.stl" />
         </xacro:if>
@@ -15,5 +15,5 @@
             <xacro:property name="upper_leg_to_lower_leg" value="${upper_leg_to_lower_leg_distance}" />
             <xacro:property name="hip_mesh_path" value="package://hyper_pupper_complete/meshes/${leg}_hip.stl" />
-            <xacro:property name="upper_leg_mesh_path" value="package://hyper_pupper_complete/meshes/${leg}_upper_leg.stl" />
+            <xacro:property name="upper_leg_mesh_path" value="package://hyper_pupper_complete/meshes/${leg}_lower_leg.stl" />
             <xacro:property name="lower_leg_mesh_path" value="package://hyper_pupper_complete/meshes/${leg}_lower_leg.stl" />
         </xacro:if>
@@ -23,5 +23,5 @@
             <xacro:property name="upper_leg_to_lower_leg" value="-${upper_leg_to_lower_leg_distance}" />
             <xacro:property name="hip_mesh_path" value="package://hyper_pupper_complete/meshes/${leg}_hip.stl" />
-            <xacro:property name="upper_leg_mesh_path" value="package://hyper_pupper_complete/meshes/${leg}_upper_leg.stl" />
+            <xacro:property name="upper_leg_mesh_path" value="package://hyper_pupper_complete/meshes/${leg}_lower_leg.stl" />
             <xacro:property name="lower_leg_mesh_path" value="package://hyper_pupper_complete/meshes/${leg}_lower_leg.stl" />
         </xacro:if>
@@ -31,5 +31,5 @@
             <xacro:property name="upper_leg_to_lower_leg" value="-${upper_leg_to_lower_leg_distance}" />
             <xacro:property name="hip_mesh_path" value="package://hyper_pupper_complete/meshes/${leg}_hip.stl" />
-            <xacro:property name="upper_leg_mesh_path" value="package://hyper_pupper_complete/meshes/${leg}_upper_leg.stl" />
+            <xacro:property name="upper_leg_mesh_path" value="package://hyper_pupper_complete/meshes/${leg}_lower_leg.stl" />
             <xacro:property name="lower_leg_mesh_path" value="package://hyper_pupper_complete/meshes/${leg}_lower_leg.stl" />
         </xacro:if>

File: src/Week04/hyper_pupper_complete/urdf/mini-pupper.urdf.xacro (robot description, xacro)
@@ -9,5 +9,5 @@
             <origin xyz="0 0 0" rpy="0 0 0" />
             <geometry>
-                <mesh filename="${base_mesh_path}" scale="1 1 1" />
+                <mesh filename="${base_mesh_path}" scale="0.001 0.001 0.001" />
             </geometry>
         </collision>
